File: Kicad/ESP32Vfo.kicad_pcb (KiCad board)
At the start: 4 copper layers, 100 x 57 mm, 127 parts, among them J1 ILI9341, J10 USB_C_Receptacle_USB2.0, J11 Link-out 1-0, J12 Link-out 1-0, J13 Link-out 1-1, J14 Link-out 1-1, J2 5V, J3 Jtag, J4 I2C, J5 Relais, J6 I2C, J7 Encoders, J8 Encoders, J9 Analog in 3-6, Q1 2N3904_SOT23, Q2 2N3904_SOT23, Q3 BFR92, Q4 BFR92, Q5 BFR92, Q6 BFR92, Q7 2N3904_SOT23, Q8 2N3904_SOT23, SW1 SW_Push, SW2 SW_Push, U1 LM1117-3.3, U2 ESP32-WROOM-32D, U3 PCF8574A, U4 CP2102N-A01-GQFN28, U5 TCA9548APWR, U6 Si5351A-B-GT, U7 Si5351A-B-GT, Y1 Crystal, Y2 Crystal

Commit message: pcb update
Routing:
- net SCL_4: track 60.3 -> 61.8 mm
- net SDA_4: track 73.3 -> 74.0 mm
Other:
- net class Default removed
